File: pantun.kicad_pcb (KiCad board)
At the start: 2 copper layers, 267.3 x 92.8 mm, 93 parts, among them J1 Conn_01x01, J2 Conn_01x01, J3 Conn_01x01, U1 promicro

Commit message: moved thumb row 1/4u to the left and added one 1u.
Parts:
- added diode40: diode, footprints:diode-sod-123, F.Cu at (114.2, 90.3)
- added switch42: switch, footprints:100-socket-solder, F.Cu at (115.9, 82.2)
- diode1, diode10, diode11, diode12, diode13, diode14, diode15, diode16, diode17, diode18, diode19, diode2, diode20, diode21, diode22, diode23, diode24, diode25, diode26, diode27, diode28, diode29, diode3, diode30, diode31, diode32, diode33, diode34, diode35, diode36, diode37, diode38, diode39, diode4, diode5, diode6, diode7, diode8, diode9: footprint Diode_SMD:D_SOD-123 -> footprints:diode-sod-123
- diode41: renamed from diode40; footprint Diode_SMD:D_SOD-123 -> footprints:diode-sod-123
- diode42: renamed from diode41; footprint Diode_SMD:D_SOD-123 -> footprints:diode-sod-123
- diode43: renamed from diode42; footprint Diode_SMD:D_SOD-123 -> footprints:diode-sod-123
- diode44: renamed from diode43; footprint Diode_SMD:D_SOD-123 -> footprints:diode-sod-123
- moved diode39 4.76 mm to (90.7, 85.3)
- moved switch39 4.76 mm to (60.0, 70.3)
- moved switch40 4.76 mm to (78.7, 74.2)
- moved switch41 4.76 mm to (97.3, 78.2)
- moved diode37 4.76 mm to (58.3, 78.4)
- moved diode38 4.76 mm to (81.8, 83.4)
- moved switch36 4.76 mm to (88.0, 76.2)
- moved diode27 2.00 mm to (74.3, 62.3)
- renumbered switch42 to switch43, switch43 to switch44, switch44 to switch45, switch45 to switch46, switch46 to switch47
Connections:
- switch36 pad 2: C6 -> C5
- switch39 pad 2: C4 -> C3
- switch40 pad 2: C5 -> C4
- switch41 pad 2: C6 -> C5
Routing:
- net C5: track 136.0 -> 169.1 mm
- net C6: track 150.9 -> 118.9 mm
- net C3: track 149.7 -> 173.1 mm
- net Net-(diode40-Pad2): track 0.00 -> 12.9 mm
- net R3: track 313.5 -> 316.4 mm
- net R4: track 377.9 -> 379.8 mm
Other:
- board text added: "berburu ke padang datar dapat rusa belang kaki berguru kepalang ajar bagai bunga kembang tak jadi"
