File: pantun.kicad_pcb (KiCad board)
At the start: 2 copper layers, 267.3 x 92.8 mm, 95 parts, among them J1 Conn_01x01, J2 Conn_01x01, J3 Conn_01x01, U1 promicro

Commit message: added led. lol.
Parts:
- added D1: LED, LED_THT:LED_D2.0mm_W4.0mm_H2.8mm_FlatTop, F.Cu at (9.39, 37.6)
- added D2: LED, LED_THT:LED_D2.0mm_W4.0mm_H2.8mm_FlatTop, F.Cu at (15.1, 75.2)
- added R1: R_Small, Resistor_THT:R_Box_L8.4mm_W2.5mm_P5.08mm, F.Cu at (97.0, 5.00)
- moved diode13 10.1 mm to (0.76, 33.3), turned to 90 degrees
- moved diode36 9.88 mm to (7.37, 71.4), turned to 90 degrees
Connections:
- U1 pad 2: unconnected-(U1-Pad2) -> Net-(U1-Pad2)
Routing:
- net GND: track 70.5 -> 292.9 mm
- net Net-(D1-Pad2): track 0.00 -> 190.4 mm
- net Net-(U1-Pad2): track 0.00 -> 39.1 mm
- net unconnected-(U1-Pad2): track 19.0 -> 0.00 mm
- net R2: track 284.1 -> 297.1 mm
- net R4: track 379.8 -> 390.0 mm
- net Net-(diode13-Pad2): track 13.0 -> 17.2 mm
- net Net-(diode36-Pad2): track 13.0 -> 16.9 mm
