File: pantun.kicad_sch (KiCad schematic)
At the start: 93 parts, among them J1 Conn_01x01, J2 Conn_01x01, J3 Conn_01x01, U1 promicro

Commit message: moved thumb row 1/4u to the left and added one 1u.
Parts:
- added diode40: diode, footprints:diode-sod-123, symbol rick-kicad-lib:diode
- added switch42: switch, footprints:100-socket-solder, symbol rick-kicad-lib:switch
- diode1, diode10, diode11, diode12, diode13, diode14, diode15, diode16, diode17, diode18, diode19, diode2, diode20, diode21, diode22, diode23, diode24, diode25, diode26, diode27, diode28, diode29, diode3, diode30, diode31, diode32, diode33, diode34, diode35, diode36, diode37, diode38, diode39, diode4, diode5, diode6, diode7, diode8, diode9: footprint Diode_SMD:D_SOD-123 -> footprints:diode-sod-123
- diode41: renamed from diode40; footprint Diode_SMD:D_SOD-123 -> footprints:diode-sod-123
- diode42: renamed from diode41; footprint Diode_SMD:D_SOD-123 -> footprints:diode-sod-123
- diode43: renamed from diode42; footprint Diode_SMD:D_SOD-123 -> footprints:diode-sod-123
- diode44: renamed from diode43; footprint Diode_SMD:D_SOD-123 -> footprints:diode-sod-123
- renumbered switch42 to switch43, switch43 to switch44, switch44 to switch45, switch45 to switch46, switch46 to switch47
Connections:
- net C3: now also switch39.2
- net C4: now also switch40.2; no longer switch39.2
- net C5: now also switch36.2, switch41.2; no longer switch40.2
- net C6: now also switch42.2; no longer switch36.2, switch41.2
- net R4: now also diode40.1
- new net: diode40.2, switch42.1
Other:
- moved on the sheet: diode37, diode38, diode39, switch36, switch39, switch40, switch41

Commit message: added led. lol.
Parts:
- added D1, D2: LED, LED_THT:LED_D2.0mm_W4.0mm_H2.8mm_FlatTop, symbol Device:LED
- added R1: R_Small, Resistor_THT:R_Box_L8.4mm_W2.5mm_P5.08mm, symbol Device:R_Small
Connections:
- net GND: now also D1.1 (K), D2.1 (K)
- net at U1.2 (RX): now also R1.2
- new net: D1.2 (A), D2.2 (A), R1.1
Changed lines of the file:
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@@
   (junction (at 232.41 28.575) (diameter 0) (color 0 0 0 0)
   )
+  (junction (at 120.015 113.03) (diameter 0) (color 0 0 0 0)
+  )
   (junction (at 191.77 60.325) (diameter 0) (color 0 0 0 0)
   )
@@
     (stroke (width 0) (type default) (color 0 0 0 0))
   )
+  (wire (pts (xy 120.015 113.03) (xy 134.62 113.03))
+    (stroke (width 0) (type default) (color 0 0 0 0))
+  )
   (wire (pts (xy 166.37 23.495) (xy 166.37 39.37))
     (stroke (width 0) (type default) (color 0 0 0 0))
@@
     (stroke (width 0) (type default) (color 0 0 0 0))
   )
+  (wire (pts (xy 120.015 115.57) (xy 120.015 113.03))
+    (stroke (width 0) (type default) (color 0 0 0 0))
+  )
   (wire (pts (xy 171.45 28.575) (xy 191.77 28.575))
     (stroke (width 0) (type default) (color 0 0 0 0))
@@
     (stroke (width 0) (type default) (color 0 0 0 0))
   )
+  (wire (pts (xy 120.015 113.03) (xy 112.395 113.03))
+    (stroke (width 0) (type default) (color 0 0 0 0))
+  )
   (wire (pts (xy 17.78 44.45) (xy 38.1 44.45))
     (stroke (width 0) (type default) (color 0 0 0 0))
@@
     (stroke (width 0) (type default) (color 0 0 0 0))
   )
+  (wire (pts (xy 139.7 113.03) (xy 156.845 113.03))
+    (stroke (width 0) (type default) (color 0 0 0 0))
+  )
   (wire (pts (xy 267.97 71.12) (xy 267.97 86.995))
     (stroke (width 0) (type default) (color 0 0 0 0))
@@
   )
   (wire (pts (xy 134.62 39.37) (xy 134.62 55.245))
+    (stroke (width 0) (type default) (color 0 0 0 0))
+  )
+  (wire (pts (xy 112.395 113.03) (xy 112.395 115.57))
     (stroke (width 0) (type default) (color 0 0 0 0))
   )
@@
     )
   )
+  (global_label "GND" (shape input) (at 120.015 123.19 270) (fields_autoplaced)
+    (effects (font (size 1.27 1.27)) (justify right))
+    (property "Intersheet References" "${INTERSHEET_REFS}" (id 0) (at 119.9356 129.4736 90)
+      (effects (font (size 1.27 1.27)) (justify right) hide)
+    )
+  )
   (global_label "R1" (shape input) (at 192.405 138.43 0) (fields_autoplaced)
     (effects (font (size 1.27 1.27)) (justify left))
@@
     (effects (font (size 1.27 1.27)) (justify right))
     (property "Intersheet References" "${INTERSHEET_REFS}" (id 0) (at 232.0833 134.5406 0)
+      (effects (font (size 1.27 1.27)) (justify right) hide)
+    )
+  )
+  (global_label "GND" (shape input) (at 112.395 123.19 270) (fields_autoplaced)
+    (effects (font (size 1.27 1.27)) (justify right))
+    (property "Intersheet References" "${INTERSHEET_REFS}" (id 0) (at 112.3156 129.4736 90)
       (effects (font (size 1.27 1.27)) (justify right) hide)
     )
@@
     (pin "2")
   )
+  (symbol (lib_id "Device:R_Small") (at 137.16 113.03 90) (unit 1)
+    (in_bom yes) (on_board yes) (fields_autoplaced)
+    (property "Reference" "R1" (id 0) (at 137.16 108.3269 90))
+    (property "Value" "R_Small" (id 1) (at 137.16 111.102 90))
+    (property "Footprint" "Resistor_THT:R_Box_L8.4mm_W2.5mm_P5.08mm" (id 2) (at 137.16 113.03 0)
+      (effects (font (size 1.27 1.27)) hide)
+    )
+    (property "Datasheet" "~" (id 3) (at 137.16 113.03 0)
+      (effects (font (size 1.27 1.27)) hide)
+    )
+    (pin "1")
+    (pin "2")
+  )
   (symbol (lib_id "rick-kicad-lib:switch") (at 219.71 23.495 0) (unit 1)
     (in_bom yes) (on_board yes) (fields_autoplaced)
@@
     (pin "2")
   )
+  (symbol (lib_id "Device:LED") (at 112.395 119.38 90) (unit 1)
+    (in_bom yes) (on_board yes) (fields_autoplaced)
+    (property "Reference" "D1" (id 0) (at 115.316 120.059 90)
+      (effects (font (size 1.27 1.27)) (justify right))
+    )
+    (property "Value" "LED" (id 1) (at 115.316 122.8341 90)
+      (effects (font (size 1.27 1.27)) (justify right))
+    )
+    (property "Footprint" "LED_THT:LED_D2.0mm_W4.0mm_H2.8mm_FlatTop" (id 2) (at 112.395 119.38 0)
+      (effects (font (size 1.27 1.27)) hide)
+    )
+    (property "Datasheet" "~" (id 3) (at 112.395 119.38 0)
+      (effects (font (size 1.27 1.27)) hide)
+    )
+    (pin "1")
+    (pin "2")
+  )
   (symbol (lib_id "rick-kicad-lib:diode") (at 232.41 27.305 180) (unit 1)
     (in_bom yes) (on_board yes) (fields_autoplaced)
@@
     (pin "2")
   )
+  (symbol (lib_id "Device:LED") (at 120.015 119.38 90) (unit 1)
+    (in_bom yes) (on_board yes) (fields_autoplaced)
+    (property "Reference" "D2" (id 0) (at 122.936 120.059 90)
+      (effects (font (size 1.27 1.27)) (justify right))
+    )
+    (property "Value" "LED" (id 1) (at 122.936 122.8341 90)
+      (effects (font (size 1.27 1.27)) (justify right))
+    )
+    (property "Footprint" "LED_THT:LED_D2.0mm_W4.0mm_H2.8mm_FlatTop" (id 2) (at 120.015 119.38 0)
+      (effects (font (size 1.27 1.27)) hide)
+    )
+    (property "Datasheet" "~" (id 3) (at 120.015 119.38 0)
+      (effects (font (size 1.27 1.27)) hide)
+    )
+    (pin "1")
+    (pin "2")
+  )
   (symbol (lib_id "rick-kicad-lib:diode") (at 38.1 43.18 180) (unit 1)
     (in_bom yes) (on_board yes) (fields_autoplaced)
@@
   )
   (symbol_instances
+    (path "/6f4ed46c-1446-402f-b1dc-8b07ca556e12"
+      (reference "D1") (unit 1) (value "LED") (footprint "LED_THT:LED_D2.0mm_W4.0mm_H2.8mm_FlatTop")
+    )
+    (path "/a3300d9e-5df3-4330-94ad-c751f1cdcdcb"
+      (reference "D2") (unit 1) (value "LED") (footprint "LED_THT:LED_D2.0mm_W4.0mm_H2.8mm_FlatTop")
+    )
     (path "/3d5e1a2f-070e-4358-9f6e-f7096c11cf5e"
       (reference "J1") (unit 1) (value "Conn_01x01") (footprint "footprints:wirepad")
@@
       (reference "J3") (unit 1) (value "Conn_01x01") (footprint "footprints:wirepad")
     )
+    (path "/638ba879-abb1-4c4e-a66c-e1b746381ba7"
+      (reference "R1") (unit 1) (value "R_Small") (footprint "Resistor_THT:R_Box_L8.4mm_W2.5mm_P5.08mm")
+    )
     (path "/0e361449-0597-45d8-951e-ba44a7567985"
